File: 001-Acorn-Electron-Plus1-GitHub/001-Acorn-Electron-Plus1.kicad_sch (KiCad schematic)
At the start: 58 parts, among them IC1 74LS30, IC10 74LS00, IC11 ADC0884, IC12 74LS195, IC13 74LS32, IC14 2764, IC15 74LS125, IC16 74LS273, IC2 74LS00, IC3 74LS139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

Commit message: V1.1 upload with all changes from Stardot and other issues found
Change 74LS260 Symbol to to a NOR Gate not a NAND gate
Change all Decoupling Caps to 100nF
Change PHI2 to PHI0
Move Left Analogue hole to line up with Molding mounting hole post
Move IC6 up 1.6mm to allow for AP6 to fit.
1 Holes missing around Cartrigde Slot
Connect IC6 pin 2 to Pin 3 IC8 - ROMQA
Tidy up some routing on the PCB
Delete ground connection on IC5 that shouldnt be there.
Parts:
- C1, C10, C13, C17, C18, C19, C20, C21, C6, C7, C8, C9: value 470pf -> 100nf
- C11, C12, C14, C16, C2: value 470pF -> 100nf
Connections:
- net ROMQA: now also IC6.2 (Q0)
- net at IC10.10, IC10.5, IC7.2: now also IC10.4, IC6.6 (~{Q1})
- net PHI2 renamed PHI0
Other:
- moved on the sheet: C2, C6, IC10B, IC10C, IC13A, IC13C, IC13D, IC1A, IC2A, IC2B, IC2C, IC2D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
